Commit message: Patch 3 -- Localization + EKF
Known Issues:
- Vector is really small in rviz.
- EKF needs to be finetuned, right now vector is just teleporting. Also I know the camera readings are jumpy so tuning might
not be only solution. Might need my outlier detection.

Signed-off-by: mihir <mihir@Vector-ROS2.myguest.virtualbox.org>

File: src/vector_description/urdf/vector.xacro (robot description, xacro)
@@ -3,5 +3,12 @@
   <!-- Inertia util -->
   <xacro:include filename="$(find vector_description)/urdf/inertia.xacro"/>
-  <link name="base_footprint"/>
+  <link name="base_footprint">
+    <visual>
+      <geometry>
+        <box size="0.001 0.001 0.001"/>
+      </geometry>
+      <material name="black"/>
+    </visual>
+  </link>
   <joint name="base_footprint_joint" type="fixed">
     <origin rpy="0 0 0" xyz="-0.01 0 0.027"/>

Commit message: Patch 5  -- Ported my previous EKF here
Working ish. Going to need to make some changes tho.

Signed-off-by: mihir <mihir@Vector-ROS2.myguest.virtualbox.org>

File: src/vector_description/urdf/vector.xacro (robot description, xacro)
@@ -3,12 +3,5 @@
   <!-- Inertia util -->
   <xacro:include filename="$(find vector_description)/urdf/inertia.xacro"/>
-  <link name="base_footprint">
-    <visual>
-      <geometry>
-        <box size="0.001 0.001 0.001"/>
-      </geometry>
-      <material name="black"/>
-    </visual>
-  </link>
+  <link name="base_footprint"/>
   <joint name="base_footprint_joint" type="fixed">
     <origin rpy="0 0 0" xyz="-0.01 0 0.027"/>
